Commit message: backup

File: install/SH_Humanoid_description/share/SH_Humanoid_description/urdf/SH_Humanoid_head.urdf (robot description, URDF)
Before this commit: robot SH_Humanoid, 16 links, 15 joints
Joints:
- joint joint1: limit effort=200.02 velocity=2.826 -> lower=-1.658063 upper=1.658063 effort=200.02 velocity=2.826; type continuous -> revolute
- joint joint10: limit effort=200.02 velocity=2.826 -> lower=-2.181662 upper=2.181662 effort=200.02 velocity=2.826; type continuous -> revolute
- joint joint11: limit effort=200.02 velocity=2.826 -> lower=-1.745329 upper=1.745329 effort=200.02 velocity=2.826; type continuous -> revolute
- joint joint12: limit effort=82.84 velocity=7.85 -> lower=-1.570796 upper=1.570796 effort=82.84 velocity=7.85; type continuous -> revolute
- joint joint13: limit effort=82.84 velocity=7.85 -> lower=-1.658063 upper=1.658063 effort=82.84 velocity=7.85; type continuous -> revolute
- joint joint14: limit effort=38.44 velocity=8.61 -> lower=-1.396263 upper=1.396263 effort=38.44 velocity=8.61; type continuous -> revolute
- joint joint2: limit effort=200.02 velocity=2.826 -> lower=-1.658063 upper=0.0 effort=200.02 velocity=2.826; type continuous -> revolute
- joint joint3: limit effort=200.02 velocity=2.826 -> lower=-2.181662 upper=2.181662 effort=200.02 velocity=2.826; type continuous -> revolute
- joint joint4: limit effort=200.02 velocity=2.826 -> lower=-1.745329 upper=1.745329 effort=200.02 velocity=2.826; type continuous -> revolute
- joint joint5: limit effort=82.84 velocity=7.85 -> lower=-1.570796 upper=1.570796 effort=82.84 velocity=7.85; type continuous -> revolute
- joint joint6: limit effort=82.84 velocity=7.85 -> lower=-1.658063 upper=1.658063 effort=82.84 velocity=7.85; type continuous -> revolute
- joint joint7: limit effort=38.44 velocity=8.61 -> lower=-1.396263 upper=1.396263 effort=38.44 velocity=8.61; type continuous -> revolute
- joint joint8: limit effort=200.02 velocity=2.826 -> lower=-1.658063 upper=1.658063 effort=200.02 velocity=2.826; type continuous -> revolute
- joint joint9: limit effort=200.02 velocity=2.826 -> lower=0.0 upper=1.658063 effort=200.02 velocity=2.826; type continuous -> revolute

Commit message: new version

File: install/SH_Humanoid_description/share/SH_Humanoid_description/urdf/SH_Humanoid_head.urdf (robot description, URDF)
Before this commit: robot SH_Humanoid, 16 links, 15 joints
Joints:
- removed joint Revolute 15
- added joint Revolute15: type continuous, parent base_link, child Head__1__1, origin xyz=0.0 0.105 0.203731 rpy=0 0 0, axis 0.0 -0.0 -1.0, limit effort=200.02 velocity=2.826
- joint joint2: limit lower=-1.658063 upper=0.0 effort=200.02 velocity=2.826 -> lower=-2.181661 upper=0.0 effort=200.02 velocity=2.826
- joint joint9: limit lower=0.0 upper=1.658063 effort=200.02 velocity=2.826 -> lower=0.0 upper=2.181661 effort=200.02 velocity=2.826

File: install/SH_moveit_limit_config/share/SH_moveit_limit_config/config/SH_Humanoid.ros2_control.xacro (robot description, xacro)
@@ -1,117 +1 @@
-<?xml version="1.0"?>
-<robot xmlns:xacro="http://www.ros.org/wiki/xacro">
-    <xacro:macro name="SH_Humanoid_ros2_control" params="name initial_positions_file">
-        <xacro:property name="initial_positions" value="${xacro.load_yaml(initial_positions_file)['initial_positions']}"/>
-        <ros2_control name="${name}" type="system">
-            <hardware>
-                <!-- By default, set up controllers for simulation. This won't work on real hardware -->
-                <plugin>mock_components/GenericSystem</plugin>
-            </hardware>
-            <joint name="joint1">
-                <command_interface name="position"/>
-                <state_interface name="position">
-                  <param name="initial_value">${initial_positions['joint1']}</param>
-                </state_interface>
-                <state_interface name="velocity"/>
-            </joint>
-            <joint name="joint2">
-                <command_interface name="position"/>
-                <state_interface name="position">
-                  <param name="initial_value">${initial_positions['joint2']}</param>
-                </state_interface>
-                <state_interface name="velocity"/>
-            </joint>
-            <joint name="joint3">
-                <command_interface name="position"/>
-                <state_interface name="position">
-                  <param name="initial_value">${initial_positions['joint3']}</param>
-                </state_interface>
-                <state_interface name="velocity"/>
-            </joint>
-            <joint name="joint4">
-                <command_interface name="position"/>
-                <state_interface name="position">
-                  <param name="initial_value">${initial_positions['joint4']}</param>
-                </state_interface>
-                <state_interface name="velocity"/>
-            </joint>
-            <joint name="joint5">
-                <command_interface name="position"/>
-                <state_interface name="position">
-                  <param name="initial_value">${initial_positions['joint5']}</param>
-                </state_interface>
-                <state_interface name="velocity"/>
-            </joint>
-            <joint name="joint6">
-                <command_interface name="position"/>
-                <state_interface name="position">
-                  <param name="initial_value">${initial_positions['joint6']}</param>
-                </state_interface>
-                <state_interface name="velocity"/>
-            </joint>
-            <joint name="joint7">
-                <command_interface name="position"/>
-                <state_interface name="position">
-                  <param name="initial_value">${initial_positions['joint7']}</param>
-                </state_interface>
-                <state_interface name="velocity"/>
-            </joint>
-            <joint name="joint8">
-                <command_interface name="position"/>
-                <state_interface name="position">
-                  <param name="initial_value">${initial_positions['joint8']}</param>
-                </state_interface>
-                <state_interface name="velocity"/>
-            </joint>
-            <joint name="joint9">
-                <command_interface name="position"/>
-                <state_interface name="position">
-                  <param name="initial_value">${initial_positions['joint9']}</param>
-                </state_interface>
-                <state_interface name="velocity"/>
-            </joint>
-            <joint name="joint10">
-                <command_interface name="position"/>
-                <state_interface name="position">
-                  <param name="initial_value">${initial_positions['joint10']}</param>
-                </state_interface>
-                <state_interface name="velocity"/>
-            </joint>
-            <joint name="joint11">
-                <command_interface name="position"/>
-                <state_interface name="position">
-                  <param name="initial_value">${initial_positions['joint11']}</param>
-                </state_interface>
-                <state_interface name="velocity"/>
-            </joint>
-            <joint name="joint12">
-                <command_interface name="position"/>
-                <state_interface name="position">
-                  <param name="initial_value">${initial_positions['joint12']}</param>
-                </state_interface>
-                <state_interface name="velocity"/>
-            </joint>
-            <joint name="joint13">
-                <command_interface name="position"/>
-                <state_interface name="position">
-                  <param name="initial_value">${initial_positions['joint13']}</param>
-                </state_interface>
-                <state_interface name="velocity"/>
-            </joint>
-            <joint name="joint14">
-                <command_interface name="position"/>
-                <state_interface name="position">
-                  <param name="initial_value">${initial_positions['joint14']}</param>
-                </state_interface>
-                <state_interface name="velocity"/>
-            </joint>
-            <joint name="Revolute15">
-                <command_interface name="position"/>
-                <state_interface name="position">
-                  <param name="initial_value">${initial_positions['Revolute15']}</param>
-                </state_interface>
-                <state_interface name="velocity"/>
-            </joint>
-        </ros2_control>
-    </xacro:macro>
-</robot>
+/home/sejong/Desktop/SH_ws/src/SH_moveit_limit_config/config/SH_Humanoid.ros2_control.xacro

File: install/SH_moveit_limit_config/share/SH_moveit_limit_config/config/SH_Humanoid.urdf.xacro (robot description, xacro)
@@ -1,9 +1 @@
-<?xml version="1.0"?>
-<robot xmlns:xacro="http://www.ros.org/wiki/xacro" name="SH_Humanoid">
-    <xacro:arg name="initial_positions_file" default="initial_positions.yaml" />
-    <!-- Import SH_Humanoid urdf file -->
-    <xacro:include filename="$(find SH_Humanoid_description)/urdf/SH_Humanoid_head.urdf" />
-    <!-- Import control_xacro -->
-    <xacro:include filename="SH_Humanoid.ros2_control.xacro" />
-    <xacro:SH_Humanoid_ros2_control name="FakeSystem" initial_positions_file="$(arg initial_positions_file)"/>
-</robot>
+/home/sejong/Desktop/SH_ws/src/SH_moveit_limit_config/config/SH_Humanoid.urdf.xacro
